Commit message: added diff drive plugin

File: description/gazebo.xacro (robot description, xacro)
@@ -12,6 +12,30 @@
     <gazebo reference="castor">
         <material>Gazebo/Blue</material>
+    </gazebo>
+    <!-- <gazebo reference="laser_frame">
+        <material>Gazebo/Red</material>
+    </gazebo> -->
+    <gazebo reference="castor">
+        <material>Gazebo/Blue</material>
         <mu1 value="0.001"/>
         <mu2 value="0.001"/>
     </gazebo>
+    <gazebo>
+        <plugin name='diff_drive' filename='libgazebo_ros_diff_drive.so'>
+            <!-- Wheel Information -->
+            <left_joint>left_wheel_joint</left_joint>
+            <right_joint>right_wheel_joint</right_joint>
+            <wheel_separation>0.36</wheel_separation>
+            <wheel_diameter>0.2</wheel_diameter>
+            <!-- Limits -->
+            <max_wheel_torque>5</max_wheel_torque>
+            <max_wheel_acceleration>2.0</max_wheel_acceleration>
+            <!-- Output -->
+            <odometry_frame>odom</odometry_frame>
+            <robot_base_frame>base_link</robot_base_frame>
+            <publish_odom>true</publish_odom>
+            <publish_odom_tf>true</publish_odom_tf>
+            <publish_wheel_tf>true</publish_wheel_tf>
+        </plugin>
+    </gazebo>
 </robot>

File: description/robot_core.urdf.xacro (robot description, xacro)
@@ -60,5 +60,5 @@
         <parent link="chassis"/>
         <child link="right_wheel"/>
-        <axis xyz="0.0 0.0 1.0"/>
+        <axis xyz="0.0 0.0 -1.0"/>
     </joint>
     <link name="right_wheel">

Commit message: added laser

File: description/gazebo.xacro (robot description, xacro)
@@ -39,3 +39,30 @@
         </plugin>
     </gazebo>
+    <gazebo reference="laser">
+        <sensor name="laser" type="ray">
+            <pose> 0 0 0 0 0 0 </pose>
+            <visualize>true</visualize>
+            <update_rate>10</update_rate>
+            <ray>
+                <scan>
+                    <horizontal>
+                        <samples>360</samples>
+                        <min_angle>-3.14</min_angle>
+                        <max_angle>3.14</max_angle>
+                    </horizontal>
+                </scan>
+                <range>
+                    <min>0.2</min>
+                    <max>5</max>
+                </range>
+            </ray>
+            <plugin name="laser_controller" filename="libgazebo_ros_ray_sensor.so">
+                <ros>
+                    <argument>~/out:=scan</argument>
+                </ros>
+                <output_type>sensor_msgs/LaserScan</output_type> <!-- baad mai explain kar dunga-->
+                <frame_name>laser</frame_name>
+            </plugin>
+        </sensor>
+    </gazebo>
 </robot>

File: description/robot_core.urdf.xacro (robot description, xacro)
@@ -108,3 +108,31 @@
         </collision>
     </link>
+    <joint name="laser_link" type="fixed">
+        <origin xyz="0.1 0.0 0.11" rpy="0.0 0.0 0.0"/>
+        <parent link="chassis"/>
+        <child link="laser"/>
+    </joint>
+    <link name="laser">
+        <xacro:inertial_box mass="0.1" x="0.1" y="0.1" z="0.03">
+            <origin xyz="0.0 0 0.0" rpy="0 0 0"/>
+        </xacro:inertial_box>
+        <visual name="">
+            <origin xyz="0.0 0.0 0.0" rpy="0.0 0.0 0.0"/>
+            <geometry>
+                <!-- <box size="0.1 0.1 0.03"/> -->
+                <cylinder radius="0.05" length="0.03"/>
+            </geometry>
+                <color rgba="1.0 0.0 0.0 0.0"/>
+            <material name="">
+                <color rgba="1.0 1.0 0.0 1.0"/>
+                <texture filename=""/>
+            </material>
+        </visual>
+        <collision>
+            <origin xyz="0.0 0.0 0.0" rpy="0.0 0.0 0.0"/>
+            <geometry>
+                <box size="0.1 0.1 0.03"/>
+            </geometry>
+        </collision>
+    </link>
 </robot>

Commit message: added camera

File: description/gazebo.xacro (robot description, xacro)
@@ -66,3 +66,43 @@
         </sensor>
     </gazebo>
+    <gazebo reference="camera">
+        <sensor type="camera" name="camera1">
+        <update_rate>30.0</update_rate>
+        <visualize>true</visualize>
+        <camera name="head">
+            <horizontal_fov>1.3962634</horizontal_fov>
+            <image>
+            <width>800</width>
+            <height>800</height>
+            <format>R8G8B8</format>
+            </image>
+            <clip>
+            <near>0.02</near>
+            <far>300</far>
+            </clip>
+            <noise>
+            <type>gaussian</type>
+            <!-- Noise is sampled independently per pixel on each frame.
+                That pixel's noise value is added to each of its color
+                channels, which at that point lie in the range [0,1]. -->
+            <mean>0.0</mean>
+            <stddev>0.007</stddev>
+            </noise>
+        </camera>
+        <plugin name="camera_controller" filename="libgazebo_ros_camera.so">
+            <alwaysOn>true</alwaysOn>
+            <updateRate>0.0</updateRate>
+            <cameraName>rrbot/camera1</cameraName>
+            <imageTopicName>image_raw</imageTopicName>
+            <cameraInfoTopicName>camera_info</cameraInfoTopicName>
+            <frameName>camera_link</frameName>
+            <hackBaseline>0.07</hackBaseline>
+            <distortionK1>0.0</distortionK1>
+            <distortionK2>0.0</distortionK2>
+            <distortionK3>0.0</distortionK3>
+            <distortionT1>0.0</distortionT1>
+            <distortionT2>0.0</distortionT2>
+        </plugin>
+        </sensor>
+  </gazebo>
 </robot>

File: description/robot_core.urdf.xacro (robot description, xacro)
@@ -114,7 +114,7 @@
     </joint>
     <link name="laser">
-        <xacro:inertial_box mass="0.1" x="0.1" y="0.1" z="0.03">
+        <xacro:inertial_cylinder mass="0.1" length="0.03" radius="0.05">
             <origin xyz="0.0 0 0.0" rpy="0 0 0"/>
-        </xacro:inertial_box>
+        </xacro:inertial_cylinder>
         <visual name="">
             <origin xyz="0.0 0.0 0.0" rpy="0.0 0.0 0.0"/>
@@ -136,3 +136,29 @@
         </collision>
     </link>
+    <joint name="camera_joint" type="fixed">
+        <origin xyz="0.15 0.0 0.07" rpy="0.0 0.0 0.0"/>
+        <parent link="chassis"/>
+        <child link="camera"/>
+    </joint>
+    <link name="camera">
+        <xacro:inertial_box mass="0.05" x="0.01" y="0.03" z="0.03">
+            <origin xyz="0.0 0 0.0" rpy="0 0 0"/>
+        </xacro:inertial_box>
+        <visual name="">
+            <origin xyz="0.0 0.0 0.0" rpy="0.0 0.0 0.0"/>
+            <geometry>
+                <box size="0.01 0.03 0.03"/>
+            </geometry>
+            <material name="">
+                <color rgba="1.0 1.0 0.0 1.0"/>
+                <texture filename=""/>
+            </material>
+        </visual>
+        <collision>
+            <origin xyz="0.0 0.0 0.0" rpy="0.0 0.0 0.0"/>
+            <geometry>
+                <box size="0.01 0.03 0.03"/>
+            </geometry>
+        </collision>
+    </link>
 </robot>
